File: rpi_breakout.sch (EAGLE design)
At the start: 21 parts

Commit message: Much nicer routing, with the help of peterobinson
Parts:
- added C3: 10uF, SparkFun:CAP_POL1206
- JP2: device SparkFun:M08LOCK -> rpi_breakout:M08LOCK
- U2, U3: device adafruit:TXB0108PWR -> rpi_breakout:TXB0108PWR
Connections:
- removed net LED3_A: LED3.A, R3.2
- removed net LED4_A: LED4.A, R4.2
- new net N$3: LED3.C, R3.1
- new net N$4: LED4.C, R4.1
- net /SPI_CE0: now also U2.A2; no longer U3.A6
- net /SPI_CE1: now also JP4.6; no longer JP3.6
- net /SPI_CEV0: now also JP4.5, U2.B2; no longer JP4.1, U3.B6
- net 3.3V: now also C1.1, C2.+, JP3.3; no longer JP3.1
- net GND: now also C3.-, JP3.2, R3.2, R4.2; no longer JP3.3, LED3.C, LED4.C
- net GPIOV_0: now also U3.B3; no longer U2.B1
- net GPIOV_1: now also U3.B2; no longer U2.B2
- net GPIOV_2: now also U3.B1; no longer U2.B3
- net GPIOV_3: now also U2.B7; no longer U2.B4
- net GPIOV_4: now also U2.B8; no longer U2.B5
- net GPIOV_6: now also U2.B4; no longer U2.B7
- net GPIOV_7: now also U3.B6; no longer U2.B8
- net GPIO_0: now also U3.A3; no longer U2.A1
- net GPIO_1: now also U3.A2; no longer U2.A2
- net GPIO_2: now also U3.A1; no longer U2.A3
- net GPIO_3: now also U2.A7; no longer U2.A4
- net GPIO_4: now also U2.A8; no longer U2.A5
- net GPIO_6: now also U2.A4; no longer U2.A7
- net GPIO_7: now also U3.A6; no longer U2.A8
- net LED3_JP: now also LED3.A; no longer R3.1
- net LED4_JP: now also LED4.A; no longer R4.1
- net RXD: now also U3.A4; no longer U3.A1
- net RXDV: now also JP4.1, U3.B4; no longer JP4.6, U3.B1
- net SPI_MISO: now also U2.A3; no longer U3.A5
- net SPI_MISOV: now also JP4.3, U2.B3; no longer JP4.2, U3.B5
- net SPI_MOSI: now also U2.A5; no longer U3.A4
- net SPI_MOSIV: now also JP4.2, U2.B5; no longer JP4.3, U3.B4
- net SPI_SCLK: now also U2.A1; no longer U3.A3
- net SPI_SCLKV: now also U2.B1; no longer U3.B3
- net TXD: now also U3.A5; no longer U3.A2
- net TXDV: now also JP3.6, U3.B5; no longer JP4.5, U3.B2
- net VCC: now also C3.+, JP3.1; no longer C1.1, C2.+, JP3.2
Other:
- moved on the sheet: C1, C2, LED3, LED4, R3, R4
