File: rpi_breakout.brd (EAGLE design)
At the start: 36.8 x 34.3 mm, 22 parts

Commit message: Oops, fix a duplicate ground connection
Routing:
- net GND: track 37.1 -> 34.4 mm
Changed lines of the file:
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@@
 <wire x1="6.5375" y1="19.685" x2="6.6675" y2="19.555" width="0.4064" layer="1"/>
 <wire x1="6.6675" y1="19.555" x2="6.6675" y2="19.05" width="0.4064" layer="1"/>
-<wire x1="6.6675" y1="19.05" x2="8.5725" y2="17.145" width="0.4064" layer="1"/>
 <wire x1="7.3025" y1="1.651" x2="7.3025" y2="2.54" width="0.4064" layer="1"/>
 <wire x1="9.8425" y1="3.81" x2="8.5725" y2="3.81" width="0.4064" layer="1"/>
@@
 <wire x1="16.35125" y1="15.875" x2="15.71625" y2="15.875" width="0.254" layer="1"/>
 <wire x1="15.71625" y1="15.875" x2="15.39875" y2="16.1925" width="0.254" layer="1"/>
-<wire x1="15.39875" y1="16.1925" x2="15.33845" y2="16.1322" width="0" layer="19" extent="1-16"/>
+<wire x1="15.39875" y1="16.1925" x2="15.33845" y2="16.1322" width="0" layer="19" extent="1-1"/>
 </signal>
 <signal name="GPIOV_3">
